File: deco-pad-v1/deco-pad-v1.sch (KiCad schematic (older format))
At the start: 86 parts, among them J1 AVR-ISP-6, SW1 EC11, SW2 EC11, SW3 EC11, SW4 SW_Push, U1 ATmega32U4-MU, U2 PRTR5VOU2X, Y1 16MHz

Commit message: [NZ] Still staging
Connections:
- net E0_PAD_A: now also SW1.A; no longer SW1.B
- net E0_PAD_B: now also SW1.B; no longer SW1.A
- net E1_PAD_A: now also SW2.A; no longer SW2.B
- net E1_PAD_B: now also SW2.B; no longer SW2.A
- net E2_PAD_A: now also SW3.A; no longer SW3.B
- net E2_PAD_B: now also SW3.B; no longer SW3.A
- net VBUS: no longer U2.4 (VCC)
- no-connect marks 9 -> 10
Changed lines of the file:
@@
 Text GLabel 1950 6100 0    50   Input ~ 0
 E2_PAD_B
+Text GLabel 4500 1350 2    50   Input ~ 0
+E0_PAD_A
 Text GLabel 4500 1150 2    50   Input ~ 0
-E0_PAD_A
-Text GLabel 4500 1350 2    50   Input ~ 0
 E0_PAD_B
-Text GLabel 4500 2050 2    50   Input ~ 0
+Text GLabel 4500 1850 2    50   Input ~ 0
 E1_PAD_B
+Text GLabel 4500 2800 2    50   Input ~ 0
+E2_PAD_A
 Text GLabel 4500 2600 2    50   Input ~ 0
-E2_PAD_A
-Text GLabel 4500 2800 2    50   Input ~ 0
 E2_PAD_B
 Wire Wire Line
@@
 	6100 2450 7000 2450
 Wire Wire Line
-	5900 2050 5900 2750
-Wire Wire Line
 	5850 2850 6150 2850
 Wire Wire Line
@@
 Wire Wire Line
 	7000 3250 6150 3250
-Wire Wire Line
-	6250 2750 5900 2750
-Connection ~ 5900 2750
-Wire Wire Line
-	5900 2750 5900 2950
 Wire Wire Line
 	7050 2350 6200 2350
@@
 Wire Notes Line
 	7450 3500 7450 1600
-Text GLabel 4500 1850 2    50   Input ~ 0
+Text GLabel 4500 2050 2    50   Input ~ 0
 E1_PAD_A
+Wire Wire Line
+	5900 2050 5900 2950
+NoConn ~ 6250 2750
 $EndSCHEMATC

Commit message: [NZ] PCB ready for review
Parts:
- removed C3, C4, C5, C6: 10n, Capacitor_SMD:C_0805_2012Metric, symbol Device:C_Small
- removed D18, D19: D_Small, Diode_SMD:D_SOD-123, symbol Device:D_Small
- removed R10, R3, R4, R5, R6, R7, R8, R9: 10K, Resistor_SMD:R_0805_2012Metric, symbol Device:R_Small
- removed SW2, SW3: EC11, Rotary_Encoder:RotaryEncoder_Alps_EC11E-Switch_Vertical_H20mm, symbol Device:Rotary_Encoder_Switch
- renumbered C14 to C10, C15 to C11, C7 to C3, C8 to C4, C9 to C5, C10 to C6, C11 to C7, C12 to C8, C13 to C9, D20 to D18, D21 to D19, R18 to R10, R19 to R11, R11 to R3, R12 to R4, R13 to R5, R14 to R6, R15 to R7, R16 to R8, R17 to R9, SW4 to SW2, U2 to U1, U1 to U2
Connections:
- net E1_PAD_A-F is gone; now on net ROW0: U2.38 (PF5)
- net E1_PAD_B-F is gone; now on net ROW1: U2.39 (PF4)
- net COL0: now also U2.29 (PB5); no longer U2.25 (PD4)
- net COL1: now also U2.28 (PB4); no longer U2.26 (PD6)
- net COL3: now also U2.26 (PD6); no longer U2.28 (PB4)
- net COL4: now also U2.25 (PD4); no longer U2.29 (PB5)
- net E0_PAD_A-F: now also C2.1
- net E0_PAD_B-F: now also C1.1
- net ROW0: no longer U2.18 (PD0)
- net ROW1: no longer U2.19 (PD1)
- net ROW2: now also U2.40 (PF1); no longer U2.20 (PD2)
- net ROW3: now also U2.41 (PF0); no longer U2.21 (PD3)
- removed net E2_PAD_A-F: C2.1, U2.40 (PF1)
- removed net E2_PAD_B-F: C1.1, U2.41 (PF0)
- no-connect marks 10 -> 14
Other:
- note added: "ENCODER_DEBOUNCE_FILTER"
- note removed: "ENCODER_DEBOUNCE_FILTERS"
- moved on the sheet: C1, C2, R1, R2, R3, R4
